File: PGA_DUAL/68882.sch (KiCad schematic (older format))
At the start: 20 parts, among them J2 MC68882_PGA, U1 74LVC1G3157

Commit message: clean-up
Parts:
- J2: DNP DNP -> (none)
Changed lines of the file:
@@
 F 5 "MPN is for a socket rather than the 68882 itself" H 3750 3600 50  0001 C CNN "Comment"
 F 6 "Layouts: https://www.precidip.com/data/files/pdf/products/pga-bga-plcc-sockets_en.pdf" H 3750 3600 50  0001 C CNN "Comment2"
-F 7 "DNP" H 3750 3600 50  0001 C CNN "DNP"
+F 7 "" H 3750 3600 50  0001 C CNN "DNP"
 	1    3750 3600
 	1    0    0    -1
