File: PGA_DUAL/IIsi.sch (KiCad schematic (older format))
At the start: 1 part, among them J1 650906-5

Commit message: clean-up
Parts:
- J1: DNP DNP -> (none)
Changed lines of the file:
@@
 F 12 "650906-5" H 4250 1075 50  0001 C CNN "MPN"
 F 13 "https://www.lcsc.com/product-detail/Mezzanine-Connectors-Board-to-Board_TE-Connectivity-650906-5_C3652939.html" H 4250 1075 50  0001 C CNN "URL"
-F 14 "DNP" H 4250 1075 50  0001 C CNN "DNP"
+F 14 "" H 4250 1075 50  0001 C CNN "DNP"
 	1    4250 1075
 	1    0    0    -1
