File: PGA_DUAL/IIsiPDSAdapter.kicad_pcb (KiCad board)
At the start: 4 copper layers, 172 x 56.7 mm, 27 parts, among them J1 650906-5, J2 MC68882_PGA, J3 5535098-5, J4 5535098-5, U1 74LVC1G3157, X1 CXO_DIP8+14

Commit message: clean-up
Parts:
- C9: value 100nF -> 100 nF
Changed lines of the file:
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@@
     (add_net GND)
+  )
+  (module For_SeeedStudio:SW_SSAJ110100 (layer F.Cu)
+    (at 85 100 180)
+    (attr smd)
+    (fp_text reference S1 (at -0.525 -3.22) (layer F.SilkS)
+      (effects (font (size 1 1) (thickness 0.15)))
+    )
+    (fp_text value SSAJ110100 (at 4.555 3.74) (layer F.Fab)
+      (effects (font (size 1 1) (thickness 0.15)))
+    )
+    (fp_poly (pts (xy -1.45255 -1.025) (xy 1.55 -1.025) (xy 1.55 0.4) (xy -1.45255 0.4)) (layer Dwgs.User) (width 0.01))
+    (fp_line (start -2.75 -1.245) (end 2.75 -1.245) (layer F.Fab) (width 0.127))
+    (fp_line (start 2.75 -1.245) (end 2.75 1.255) (layer F.Fab) (width 0.127))
+    (fp_line (start 2.75 1.255) (end 1.3 1.255) (layer F.Fab) (width 0.127))
+    (fp_line (start 1.3 1.255) (end 0.1 1.255) (layer F.Fab) (width 0.127))
+    (fp_line (start 0.1 1.255) (end -2.75 1.255) (layer F.Fab) (width 0.127))
+    (fp_line (start -2.75 1.255) (end -2.75 -1.245) (layer F.Fab) (width 0.127))
+    (fp_line (start 0.1 1.255) (end 0.1 2.355) (layer F.Fab) (width 0.127))
+    (fp_line (start 0.1 2.355) (end 0.3 2.555) (layer F.Fab) (width 0.127))
+    (fp_line (start 0.3 2.555) (end 1.1 2.555) (layer F.Fab) (width 0.127))
+    (fp_line (start 1.1 2.555) (end 1.3 2.355) (layer F.Fab) (width 0.127))
+    (fp_line (start 1.3 2.355) (end 1.3 1.255) (layer F.Fab) (width 0.127))
+    (fp_line (start -2.75 -1.245) (end -1.62 -1.245) (layer F.SilkS) (width 0.127))
+    (fp_line (start 1.62 -1.245) (end 2.75 -1.245) (layer F.SilkS) (width 0.127))
+    (fp_line (start 2.75 -1.245) (end 2.75 -0.595) (layer F.SilkS) (width 0.127))
+    (fp_line (start 2.75 1.255) (end 2.75 0.745) (layer F.SilkS) (width 0.127))
+    (fp_line (start -2.75 -0.595) (end -2.75 -1.245) (layer F.SilkS) (width 0.127))
+    (fp_line (start -2.75 1.255) (end -2.75 0.745) (layer F.SilkS) (width 0.127))
+    (fp_line (start 2.75 1.255) (end 1.3 1.255) (layer F.SilkS) (width 0.127))
+    (fp_line (start 1.3 1.255) (end 0.1 1.255) (layer F.SilkS) (width 0.127))
+    (fp_line (start 0.1 1.255) (end -2.75 1.255) (layer F.SilkS) (width 0.127))
+    (fp_line (start 0.1 1.255) (end 0.1 2.355) (layer F.SilkS) (width 0.127))
+    (fp_line (start 0.1 2.355) (end 0.3 2.555) (layer F.SilkS) (width 0.127))
+    (fp_line (start 0.3 2.555) (end 1.1 2.555) (layer F.SilkS) (width 0.127))
+    (fp_line (start 1.1 2.555) (end 1.3 2.355) (layer F.SilkS) (width 0.127))
+    (fp_line (start 1.3 2.355) (end 1.3 1.255) (layer F.SilkS) (width 0.127))
+    (fp_line (start -3.7 -1.785) (end -3.7 2.805) (layer F.CrtYd) (width 0.05))
+    (fp_line (start -3.7 2.805) (end 3.7 2.805) (layer F.CrtYd) (width 0.05))
+    (fp_line (start 3.7 2.805) (end 3.7 -1.785) (layer F.CrtYd) (width 0.05))
+    (fp_line (start 3.7 -1.785) (end -3.7 -1.785) (layer F.CrtYd) (width 0.05))
+    (fp_circle (center -1 -2.135) (end -0.9 -2.135) (layer F.SilkS) (width 0.2))
+    (fp_circle (center -1 -2.135) (end -0.9 -2.135) (layer F.Fab) (width 0.2))
+    (pad None np_thru_hole circle (at 1.5 0 180) (size 0.8 0.8) (drill 0.8) (layers *.Cu *.Mask))
+    (pad None np_thru_hole circle (at -1.5 0 180) (size 0.8 0.8) (drill 0.8) (layers *.Cu *.Mask))
+    (pad S2 smd rect (at -3 0.075 180) (size 0.9 0.7) (layers F.Cu F.Paste F.Mask))
+    (pad S1 smd rect (at 3 0.075 180) (size 0.9 0.7) (layers F.Cu F.Paste F.Mask))
+    (pad 1 smd rect (at -1 -1.28 180) (size 0.6 0.51) (layers F.Cu F.Paste F.Mask)
+      (net 114 "Net-(R5-Pad2)"))
+    (pad C smd rect (at 0 -1.28 180) (size 0.6 0.51) (layers F.Cu F.Paste F.Mask)
+      (net 115 clk_ctrl))
+    (pad 2 smd rect (at 1 -1.28 180) (size 0.6 0.51) (layers F.Cu F.Paste F.Mask)
+      (net 113 "Net-(R4-Pad2)"))
   )
   (module For_SeeedStudio:5535098-5 (layer F.Cu)
     (at 214.12 125.8)
+    (attr smd)
     (fp_text reference J4 (at -49.53 2.54) (layer F.SilkS)
       (effects (font (size 1 1) (thickness 0.15)))
@@
       (net 108 ~RBV))
   )
-  (module For_SeeedStudio:SW_SSAJ110100 (layer F.Cu)
-    (at 85 100 180)
-    (attr smd)
-    (fp_text reference S1 (at -0.525 -3.22) (layer F.SilkS)
-      (effects (font (size 1 1) (thickness 0.15)))
-    )
-    (fp_text value SSAJ110100 (at 4.555 3.74) (layer F.Fab)
-      (effects (font (size 1 1) (thickness 0.15)))
-    )
-    (fp_circle (center -1 -2.135) (end -0.9 -2.135) (layer F.Fab) (width 0.2))
-    (fp_circle (center -1 -2.135) (end -0.9 -2.135) (layer F.SilkS) (width 0.2))
-    (fp_line (start 3.7 -1.785) (end -3.7 -1.785) (layer F.CrtYd) (width 0.05))
-    (fp_line (start 3.7 2.805) (end 3.7 -1.785) (layer F.CrtYd) (width 0.05))
-    (fp_line (start -3.7 2.805) (end 3.7 2.805) (layer F.CrtYd) (width 0.05))
-    (fp_line (start -3.7 -1.785) (end -3.7 2.805) (layer F.CrtYd) (width 0.05))
-    (fp_line (start 1.3 2.355) (end 1.3 1.255) (layer F.SilkS) (width 0.127))
-    (fp_line (start 1.1 2.555) (end 1.3 2.355) (layer F.SilkS) (width 0.127))
-    (fp_line (start 0.3 2.555) (end 1.1 2.555) (layer F.SilkS) (width 0.127))
-    (fp_line (start 0.1 2.355) (end 0.3 2.555) (layer F.SilkS) (width 0.127))
-    (fp_line (start 0.1 1.255) (end 0.1 2.355) (layer F.SilkS) (width 0.127))
-    (fp_line (start 0.1 1.255) (end -2.75 1.255) (layer F.SilkS) (width 0.127))
-    (fp_line (start 1.3 1.255) (end 0.1 1.255) (layer F.SilkS) (width 0.127))
-    (fp_line (start 2.75 1.255) (end 1.3 1.255) (layer F.SilkS) (width 0.127))
-    (fp_line (start -2.75 1.255) (end -2.75 0.745) (layer F.SilkS) (width 0.127))
-    (fp_line (start -2.75 -0.595) (end -2.75 -1.245) (layer F.SilkS) (width 0.127))
-    (fp_line (start 2.75 1.255) (end 2.75 0.745) (layer F.SilkS) (width 0.127))
-    (fp_line (start 2.75 -1.245) (end 2.75 -0.595) (layer F.SilkS) (width 0.127))
-    (fp_line (start 1.62 -1.245) (end 2.75 -1.245) (layer F.SilkS) (width 0.127))
-    (fp_line (start -2.75 -1.245) (end -1.62 -1.245) (layer F.SilkS) (width 0.127))
-    (fp_line (start 1.3 2.355) (end 1.3 1.255) (layer F.Fab) (width 0.127))
-    (fp_line (start 1.1 2.555) (end 1.3 2.355) (layer F.Fab) (width 0.127))
-    (fp_line (start 0.3 2.555) (end 1.1 2.555) (layer F.Fab) (width 0.127))
-    (fp_line (start 0.1 2.355) (end 0.3 2.555) (layer F.Fab) (width 0.127))
-    (fp_line (start 0.1 1.255) (end 0.1 2.355) (layer F.Fab) (width 0.127))
-    (fp_line (start -2.75 1.255) (end -2.75 -1.245) (layer F.Fab) (width 0.127))
-    (fp_line (start 0.1 1.255) (end -2.75 1.255) (layer F.Fab) (width 0.127))
-    (fp_line (start 1.3 1.255) (end 0.1 1.255) (layer F.Fab) (width 0.127))
-    (fp_line (start 2.75 1.255) (end 1.3 1.255) (layer F.Fab) (width 0.127))
-    (fp_line (start 2.75 -1.245) (end 2.75 1.255) (layer F.Fab) (width 0.127))
-    (fp_line (start -2.75 -1.245) (end 2.75 -1.245) (layer F.Fab) (width 0.127))
-    (fp_poly (pts (xy -1.45255 -1.025) (xy 1.55 -1.025) (xy 1.55 0.4) (xy -1.45255 0.4)) (layer Dwgs.User) (width 0.01))
-    (pad None np_thru_hole circle (at 1.5 0 180) (size 0.8 0.8) (drill 0.8) (layers *.Cu *.Mask))
-    (pad None np_thru_hole circle (at -1.5 0 180) (size 0.8 0.8) (drill 0.8) (layers *.Cu *.Mask))
-    (pad S2 smd rect (at -3 0.075 180) (size 0.9 0.7) (layers F.Cu F.Paste F.Mask))
-    (pad S1 smd rect (at 3 0.075 180) (size 0.9 0.7) (layers F.Cu F.Paste F.Mask))
-    (pad 1 smd rect (at -1 -1.28 180) (size 0.6 0.51) (layers F.Cu F.Paste F.Mask)
-      (net 114 "Net-(R5-Pad2)"))
-    (pad C smd rect (at 0 -1.28 180) (size 0.6 0.51) (layers F.Cu F.Paste F.Mask)
-      (net 115 clk_ctrl))
-    (pad 2 smd rect (at 1 -1.28 180) (size 0.6 0.51) (layers F.Cu F.Paste F.Mask)
-      (net 113 "Net-(R4-Pad2)"))
-  )
   (module Capacitor_SMD:C_0603_1608Metric (layer F.Cu)
     (at 86.62 109.1 90)
@@
   (module For_SeeedStudio:MC68882_PGA locked (layer F.Cu)
     (at 79 126.25 180)
+    (attr smd)
     (fp_text reference J2 (at -14.55 -12.51) (layer F.SilkS)
       (effects (font (size 1 1) (thickness 0.15)))
@@
       (effects (font (size 1 1) (thickness 0.15)))
     )
-    (fp_text value 100nF (at 0 1.43 90) (layer F.Fab)
+    (fp_text value "100 nF" (at 0 1.43 90) (layer F.Fab)
       (effects (font (size 1 1) (thickness 0.15)))
     )
@@
     (descr 650906-5-1)
     (tags Connector)
+    (attr smd)
     (fp_text reference J1 (at -49.53 3.379) (layer F.SilkS)
       (effects (font (size 1.27 1.27) (thickness 0.254)))
@@
   (module For_SeeedStudio:5535098-5 (layer F.Cu)
     (at 203.95 100.3)
+    (attr smd)
     (fp_text reference J3 (at -48.95 10.7) (layer F.SilkS)
       (effects (font (size 1 1) (thickness 0.15)))
