File: PGA_DUAL/PDS.sch (KiCad schematic (older format))
At the start: 2 parts, among them J3 5535098-5, J4 5535098-5

Commit message: clean-up
Parts:
- J3, J4: DNP DNP -> (none); MPN (none) -> 5535098-5
Changed lines of the file:
@@
 F 10 "5535098-5" H 2675 350 50  0001 L CNN "Arrow Part Number"
 F 11 "https://www.arrow.com/en/products/5535098-5/te-connectivity" H 2675 250 50  0001 L CNN "Arrow Price/Stock"
-F 12 "DNP" H 1825 1050 50  0001 C CNN "DNP"
+F 12 "" H 1825 1050 50  0001 C CNN "DNP"
+F 13 "5535098-5" H 1825 1050 50  0001 C CNN "MPN"
 	1    1825 1050
 	1    0    0    -1
@@
 F 10 "5535098-5" H 5300 350 50  0001 L CNN "Arrow Part Number"
 F 11 "https://www.arrow.com/en/products/5535098-5/te-connectivity" H 5300 250 50  0001 L CNN "Arrow Price/Stock"
-F 12 "DNP" H 4450 1050 50  0001 C CNN "DNP"
+F 12 "" H 4450 1050 50  0001 C CNN "DNP"
+F 13 "5535098-5" H 4450 1050 50  0001 C CNN "MPN"
 	1    4450 1050
 	1    0    0    -1
