File: PGA_DUAL/clock.sch (KiCad schematic (older format))
At the start: 4 parts, among them X1 CXO_DIP8+14

Commit message: clean-up
Parts:
- C11: value 100nF -> 100 nF
Changed lines of the file:
@@
 AR Path="/6424DB31/64F9279B" Ref="C9"  Part="1"
 F 0 "C9" H 3200 2700 50  0000 L CNN
-F 1 "100nF" H 3200 2500 50  0000 L CNN
+F 1 "100 nF" H 3200 2500 50  0000 L CNN
 F 2 "Capacitor_SMD:C_0603_1608Metric" H 3213 2450 50  0001 C CNN
 F 3 "" H 3175 2600 50  0000 C CNN
